Commit message: Gazebo Yarp Plugins fixed

File: 2r_manipulator_scaled_down/model.urdf (robot description, URDF)
Before this commit: robot 2r_manipulator_scaled_down, 5 links, 4 joints
Joints:
- joint first_joint: limit lower=-0.785 upper=0.785 effort=30 velocity=1.0 -> lower=-1.57 upper=0.3925 effort=30 velocity=1.0
- joint second_joint: limit lower=-0.785 upper=0.785 effort=30 velocity=1.0 -> lower=-0.3925 upper=0.3925 effort=30 velocity=1.0

File: 2r_manipulator_scaled_down/model.xacro (robot description, xacro)
@@ -327,3 +327,8 @@
   <safety_controller k_velocity="10" k_position="15" soft_lower_limit="-1.5" soft_upper_limit="1.5"/>
 </joint>
+<!--Gazebo Yarp Plugin-->
+<!--plugin name="controlboard" filename="libgazebo_yarp_controlboard.so">
+       <yarpConfigurationFile>model://manipulator2r/conf/gazebo_controlboard.ini</yarpConfigurationFile>
+       <initialConfiguration>0.0 0.0</initialConfiguration>
+     </plugin-->
 </robot>

Commit message: fixed all axes frame to be planar

File: 2r_manipulator_scaled_down/model.urdf (robot description, URDF)
Before this commit: robot 2r_manipulator_scaled_down, 5 links, 4 joints
Joints:
- joint first_joint: limit lower=-1.57 upper=0.3925 effort=30 velocity=1.0 -> lower=-0.785 upper=0 effort=30 velocity=1.0; origin xyz=0 0.075 0.00625 rpy=0 0 0.785 -> xyz=0 0.075 0 rpy=0 0 0.3925
- joint handle_joint: origin xyz=0 0.3 -0.00625 rpy=0 0 0 -> xyz=0 0.3 0 rpy=0 0 0
- joint second_joint: origin xyz=0 0.3 0.00625 rpy=0 0 -1.57 -> xyz=0 0.3 0 rpy=0 0 -0.3925

File: 2r_manipulator_scaled_down/model.xacro (robot description, xacro)
@@ -94,5 +94,5 @@
 <link name="first_link">
   <inertial>
-    <origin xyz="0 ${radius_small_cylinder*3/2+length_small_box*3/2+length_link1_box/2} -${height_base_box/8}" rpy="0 0 0"/>
+    <origin xyz="0 ${radius_small_cylinder*3/2+length_small_box*3/2+length_link1_box/2} 0" rpy="0 0 0"/>
     <mass value="1" />
     <inertia ixx="0.1" iyy="0.1" izz="0.1" ixy="0" ixz="0" iyz="0" />
@@ -100,14 +100,14 @@
 <!--First Link Small Cylinder - Front -->
   <visual>
-    <origin xyz="0 0 ${height_base_box/8}" rpy="0 0 ${angle/4}"/>
-    <geometry>
-      <cylinder length="${length_small_cylinder}" radius="${radius_small_cylinder}"/>
-      <material name="white">
-        <color rgba="1.0 1.0 1.0 1.0"/>
-      </material>
-    </geometry>
-  </visual>
-  <collision>
-    <origin xyz="0 0 ${height_base_box/8}" rpy="0 0 ${angle/4}"/>
+    <origin xyz="0 0 ${height_base_box/4}" rpy="0 0 0"/>
+    <geometry>
+      <cylinder length="${length_small_cylinder}" radius="${radius_small_cylinder}"/>
+      <material name="white">
+        <color rgba="1.0 1.0 1.0 1.0"/>
+      </material>
+    </geometry>
+  </visual>
+  <collision>
+    <origin xyz="0 0 ${height_base_box/4}" rpy="0 0 0"/>
     <geometry>
       <cylinder length="${length_small_cylinder}" radius="${radius_small_cylinder}"/>
@@ -116,14 +116,14 @@
 <!--First Link Small Box - Front -->
   <visual>
-    <origin xyz="0 ${radius_small_cylinder*2} ${height_base_box/8}" rpy="0 0 0"/>
-    <geometry>
-      <box size="${length_small_box} ${width_small_box} ${height_small_box}"/>
-      <material name="white">
-        <color rgba="1.0 1.0 1.0 1.0"/>
-      </material>
-    </geometry>
-  </visual>
-  <collision>
-    <origin xyz="0 ${radius_small_cylinder*2} ${height_base_box/8}" rpy="0 0 0"/>
+    <origin xyz="0 ${radius_small_cylinder*2} ${height_base_box/4}" rpy="0 0 0"/>
+    <geometry>
+      <box size="${length_small_box} ${width_small_box} ${height_small_box}"/>
+      <material name="white">
+        <color rgba="1.0 1.0 1.0 1.0"/>
+      </material>
+    </geometry>
+  </visual>
+  <collision>
+    <origin xyz="0 ${radius_small_cylinder*2} ${height_base_box/4}" rpy="0 0 0"/>
     <geometry>
       <box size="${length_small_box} ${width_small_box} ${height_small_box}"/>
@@ -132,5 +132,5 @@
 <!--First Link Box-->
   <visual>
-    <origin xyz="0 ${radius_small_cylinder*6} -${height_link1_box/8}" rpy="0 0 0"/>
+    <origin xyz="0 ${radius_small_cylinder*6} 0" rpy="0 0 0"/>
     <geometry>
       <box size="${length_link1_box} ${width_link1_box} ${height_link1_box}"/>
@@ -141,5 +141,5 @@
   </visual>
   <collision>
-    <origin xyz="0 ${radius_small_cylinder*6} -${height_link1_box/8}" rpy="0 0 0"/>
+    <origin xyz="0 ${radius_small_cylinder*6} 0" rpy="0 0 0"/>
     <geometry>
       <box size="${length_link1_box} ${width_link1_box} ${height_link1_box}"/>
@@ -148,14 +148,14 @@
 <!--First Link Small Box - Back -->
   <visual>
-    <origin xyz="0 ${radius_small_cylinder*2+width_link1_box} -${height_base_box*(3/8)}" rpy="0 0 0"/>
-    <geometry>
-      <box size="${length_small_box} ${width_small_box} ${height_small_box}"/>
-      <material name="white">
-        <color rgba="1.0 1.0 1.0 1.0"/>
-      </material>
-    </geometry>
-  </visual>
-  <collision>
-    <origin xyz="0 ${radius_small_cylinder*2+width_link1_box} -${height_base_box*(3/8)}" rpy="0 0 0"/>
+    <origin xyz="0 ${radius_small_cylinder*2+width_link1_box} -${height_base_box/4}" rpy="0 0 0"/>
+    <geometry>
+      <box size="${length_small_box} ${width_small_box} ${height_small_box}"/>
+      <material name="white">
+        <color rgba="1.0 1.0 1.0 1.0"/>
+      </material>
+    </geometry>
+  </visual>
+  <collision>
+    <origin xyz="0 ${radius_small_cylinder*2+width_link1_box} -${height_base_box/4}" rpy="0 0 0"/>
     <geometry>
       <box size="${length_small_box} ${width_small_box} ${height_small_box}"/>
@@ -164,14 +164,14 @@
 <!--First Link Small Cylinder - Back -->
   <visual>
-    <origin xyz="0 ${radius_small_cylinder*4+width_link1_box} -${height_base_box*(3/8)}" rpy="0 0 0"/>
-    <geometry>
-      <cylinder length="${length_small_cylinder}" radius="${radius_small_cylinder}"/>
-      <material name="white">
-        <color rgba="1.0 1.0 1.0 1.0"/>
-      </material>
-    </geometry>
-  </visual>
-  <collision>
-    <origin xyz="0 ${radius_small_cylinder*4+width_link1_box} -${height_base_box*(3/8)}" rpy="0 0 0"/>
+    <origin xyz="0 ${radius_small_cylinder*4+width_link1_box} -${height_base_box/4}" rpy="0 0 0"/>
+    <geometry>
+      <cylinder length="${length_small_cylinder}" radius="${radius_small_cylinder}"/>
+      <material name="white">
+        <color rgba="1.0 1.0 1.0 1.0"/>
+      </material>
+    </geometry>
+  </visual>
+  <collision>
+    <origin xyz="0 ${radius_small_cylinder*4+width_link1_box} -${height_base_box/4}" rpy="0 0 0"/>
     <geometry>
       <cylinder length="${length_small_cylinder}" radius="${radius_small_cylinder}"/>
@@ -182,5 +182,5 @@
 <link name="second_link">
   <inertial>
-    <origin xyz="0 ${radius_small_cylinder*3/2+length_small_box*3/2+length_link1_box/2} -${height_base_box/4}" rpy="0 0 0"/>
+    <origin xyz="0 ${radius_small_cylinder*3/2+length_small_box*3/2+length_link1_box/2} 0" rpy="0 0 0"/>
     <mass value="1" />
     <inertia ixx="0.1" iyy="0.1" izz="0.1" ixy="0" ixz="0" iyz="0" />
@@ -188,14 +188,14 @@
 <!--Second Link Small Cylinder - Front -->
   <visual>
-    <origin xyz="0 0 0" rpy="0 0 0"/>
-    <geometry>
-      <cylinder length="${length_small_cylinder}" radius="${radius_small_cylinder}"/>
-      <material name="white">
-        <color rgba="1.0 1.0 1.0 1.0"/>
-      </material>
-    </geometry>
-  </visual>
-  <collision>
-    <origin xyz="0 0 0" rpy="0 0 0"/>
+    <origin xyz="0 0 ${height_base_box/4}" rpy="0 0 0"/>
+    <geometry>
+      <cylinder length="${length_small_cylinder}" radius="${radius_small_cylinder}"/>
+      <material name="white">
+        <color rgba="1.0 1.0 1.0 1.0"/>
+      </material>
+    </geometry>
+  </visual>
+  <collision>
+    <origin xyz="0 0 ${height_base_box/4}" rpy="0 0 0"/>
     <geometry>
       <cylinder length="${length_small_cylinder}" radius="${radius_small_cylinder}"/>
@@ -204,14 +204,14 @@
 <!--Second Link Small Box - Front -->
   <visual>
-    <origin xyz="0 ${radius_small_cylinder*2} 0" rpy="0 0 0"/>
-    <geometry>
-      <box size="${length_small_box} ${width_small_box} ${height_small_box}"/>
-      <material name="white">
-        <color rgba="1.0 1.0 1.0 1.0"/>
-      </material>
-    </geometry>
-  </visual>
-  <collision>
-    <origin xyz="0 ${radius_small_cylinder*2} 0" rpy="0 0 0"/>
+    <origin xyz="0 ${radius_small_cylinder*2} ${height_base_box/4}" rpy="0 0 0"/>
+    <geometry>
+      <box size="${length_small_box} ${width_small_box} ${height_small_box}"/>
+      <material name="white">
+        <color rgba="1.0 1.0 1.0 1.0"/>
+      </material>
+    </geometry>
+  </visual>
+  <collision>
+    <origin xyz="0 ${radius_small_cylinder*2} ${height_base_box/4}" rpy="0 0 0"/>
     <geometry>
       <box size="${length_small_box} ${width_small_box} ${height_small_box}"/>
@@ -220,5 +220,5 @@
 <!--Second Link Box-->
   <visual>
-    <origin xyz="0 ${radius_small_cylinder*6} -${height_link2_box/4}" rpy="0 0 0"/>
+    <origin xyz="0 ${radius_small_cylinder*6} 0" rpy="0 0 0"/>
     <geometry>
       <box size="${length_link2_box} ${width_link2_box} ${height_link2_box}"/>
@@ -229,5 +229,5 @@
   </visual>
   <collision>
-    <origin xyz="0 ${radius_small_cylinder*6} -${height_link2_box/4}" rpy="0 0 0"/>
+    <origin xyz="0 ${radius_small_cylinder*6} 0" rpy="0 0 0"/>
     <geometry>
       <box size="${length_link2_box} ${width_link2_box} ${height_link2_box}"/>
@@ -236,14 +236,14 @@
 <!--Second Link Small Box - Back -->
   <visual>
-    <origin xyz="0 ${radius_small_cylinder*2+width_link2_box} -${height_base_box/4+height_link2_box/4}" rpy="0 0 0"/>
-    <geometry>
-      <box size="${length_small_box} ${width_small_box} ${height_small_box}"/>
-      <material name="white">
-        <color rgba="1.0 1.0 1.0 1.0"/>
-      </material>
-    </geometry>
-  </visual>
-  <collision>
-    <origin xyz="0 ${radius_small_cylinder*2+width_link2_box} -${height_base_box/4+height_link2_box/4}" rpy="0 0 0"/>
+    <origin xyz="0 ${radius_small_cylinder*2+width_link2_box} -${height_base_box/4}" rpy="0 0 0"/>
+    <geometry>
+      <box size="${length_small_box} ${width_small_box} ${height_small_box}"/>
+      <material name="white">
+        <color rgba="1.0 1.0 1.0 1.0"/>
+      </material>
+    </geometry>
+  </visual>
+  <collision>
+    <origin xyz="0 ${radius_small_cylinder*2+width_link2_box} -${height_base_box/4}" rpy="0 0 0"/>
     <geometry>
       <box size="${length_small_box} ${width_small_box} ${height_small_box}"/>
@@ -252,14 +252,14 @@
 <!--Second Link Small Cylinder - Back -->
   <visual>
-    <origin xyz="0 ${radius_small_cylinder*4+width_link2_box} -${height_base_box/4+height_link2_box/4}" rpy="0 0 0"/>
-    <geometry>
-      <cylinder length="${length_small_cylinder}" radius="${radius_small_cylinder}"/>
-      <material name="white">
-        <color rgba="1.0 1.0 1.0 1.0"/>
-      </material>
-    </geometry>
-  </visual>
-  <collision>
-    <origin xyz="0 ${radius_small_cylinder*4+width_link2_box} -${height_base_box/4+height_link2_box/4}" rpy="0 0 0"/>
+    <origin xyz="0 ${radius_small_cylinder*4+width_link2_box} -${height_base_box/4}" rpy="0 0 0"/>
+    <geometry>
+      <cylinder length="${length_small_cylinder}" radius="${radius_small_cylinder}"/>
+      <material name="white">
+        <color rgba="1.0 1.0 1.0 1.0"/>
+      </material>
+    </geometry>
+  </visual>
+  <collision>
+    <origin xyz="0 ${radius_small_cylinder*4+width_link2_box} -${height_base_box/4}" rpy="0 0 0"/>
     <geometry>
       <cylinder length="${length_small_cylinder}" radius="${radius_small_cylinder}"/>
@@ -300,9 +300,9 @@
   <parent link="base_link"/>
   <child link="first_link"/>
-  <origin xyz="0 ${width_small_box*(3/4)} ${height_base_box/8}" rpy="0 0 ${angle/4}" />
+  <origin xyz="0 ${width_small_box*(3/4)} 0" rpy="0 0 ${angle/8}" />
   <axis xyz="0 0 1" />
   <calibration rising="1"/>
   <dynamic damping="0.0" friction="0.0"/>
-  <limit effort="30" lower="-${angle/2}" upper="${angle/8}" velocity="1.0"/>
+  <limit effort="30" lower="-${angle/4}" upper="0" velocity="1.0"/>
   <safety_controller k_velocity="10" k_position="15" soft_lower_limit="-1.5" soft_upper_limit="1.5"/>
 </joint>
@@ -310,5 +310,5 @@
   <parent link="first_link"/>
   <child link="second_link"/>
-  <origin xyz="0 ${width_small_box+width_link1_box} ${height_base_box/8}" rpy="0 0 -${angle/2}" />
+  <origin xyz="0 ${width_small_box+width_link1_box} 0" rpy="0 0 -${angle/8}" />
   <axis xyz="0 0 1" />
   <calibration rising="1"/>
@@ -320,5 +320,5 @@
   <parent link="second_link"/>
   <child link="handle_link"/>
-  <origin xyz="0 ${width_small_box+width_link2_box} -${height_base_box/8}" rpy="0 0 0" />
+  <origin xyz="0 ${width_small_box+width_link2_box} 0" rpy="0 0 0" />
   <axis xyz="0 0 1" />
   <calibration rising="1"/>
@@ -326,9 +326,17 @@
   <limit effort="30" lower="-${angle}" upper="${angle}" velocity="1.0"/>
   <safety_controller k_velocity="10" k_position="15" soft_lower_limit="-1.5" soft_upper_limit="1.5"/>
+  <!--sensor name='left_leg_ft' type='force_torque'>
+    <always_on>1</always_on>
+    <update_rate>100</update_rate>
+    <pose>0 0 0 0 0 0</pose>
+    <plugin name='handle_ft' filename='libgazebo_yarp_forcetorque.so'>
+      <yarpConfigurationFile>model://icub/conf/FT/gazebo_forcetorque.ini</yarpConfigurationFile>
+    </plugin>
+  </sensor-->
 </joint>
 <!--Gazebo Yarp Plugin-->
 <!--plugin name="controlboard" filename="libgazebo_yarp_controlboard.so">
-       <yarpConfigurationFile>model://manipulator2r/conf/gazebo_controlboard.ini</yarpConfigurationFile>
-       <initialConfiguration>0.0 0.0</initialConfiguration>
-     </plugin-->
+  <yarpConfigurationFile>model://2r_manipulator_scaled_down/conf/gazebo_controlboard.ini</yarpConfigurationFile>
+  <initialConfiguration>0.0 0.0</initialConfiguration>
+</plugin-->
 </robot>
