Commit message: set joint angles

File: 2r_manipulator_scaled_down/model.xacro (robot description, xacro)
@@ -304,5 +304,5 @@
   <calibration rising="1"/>
   <dynamic damping="0.0" friction="0.0"/>
-  <limit effort="30" lower="-${angle/4}" upper="${angle/4}" velocity="1.0"/>
+  <limit effort="30" lower="-${angle/2}" upper="${angle/8}" velocity="1.0"/>
   <safety_controller k_velocity="10" k_position="15" soft_lower_limit="-1.5" soft_upper_limit="1.5"/>
 </joint>
@@ -314,5 +314,5 @@
   <calibration rising="1"/>
   <dynamic damping="0.0" friction="0.0"/>
-  <limit effort="30" lower="-${angle/4}" upper="${angle/4}" velocity="1.0"/>
+  <limit effort="30" lower="-${angle/8}" upper="${angle/8}" velocity="1.0"/>
   <safety_controller k_velocity="10" k_position="15" soft_lower_limit="-1.5" soft_upper_limit="1.5"/>
 </joint>

Commit message: Xacro for Inertial Params

File: 2r_manipulator_scaled_down/model.xacro (robot description, xacro)
@@ -34,4 +34,22 @@
 <xacro:property name="length_handle_cylinder" value="${height_small_box*4}"/>
 <xacro:property name="radius_handle_cylinder" value="${length_small_box/4}"/>
+<!--XACRO: Link Masses-->
+<xacro:property name="base_link_mass" value="1"/>
+<xacro:property name="first_link_mass" value="1"/>
+<xacro:property name="second_link_mass" value="1"/>
+<xacro:property name="handle_link_mass" value="1"/>
+<!--XACRO: Link Inertia Value-->
+<xacro:property name="base_link_inertia_xx" value="1"/>
+<xacro:property name="base_link_inertia_yy" value="1"/>
+<xacro:property name="base_link_inertia_zz" value="1"/>
+<xacro:property name="first_link_inertia_xx" value="1"/>
+<xacro:property name="first_link_inertia_yy" value="1"/>
+<xacro:property name="first_link_inertia_zz" value="1"/>
+<xacro:property name="second_link_inertia_xx" value="1"/>
+<xacro:property name="second_link_inertia_yy" value="1"/>
+<xacro:property name="second_link_inertia_zz" value="1"/>
+<xacro:property name="handle_link_inertia_xx" value="1"/>
+<xacro:property name="handle_link_inertia_yy" value="1"/>
+<xacro:property name="handle_link_inertia_zz" value="1"/>
 <link name="world" />
 <!--Base Link is at the Origin-->
@@ -39,6 +57,6 @@
   <inertial>
     <origin xyz="0 0 0" rpy="0 0 0"/>
-    <mass value="1" />
-    <inertia ixx="0.1" iyy="0.1" izz="0.1" ixy="0" ixz="0" iyz="0" />
+    <mass value="${base_link_mass}" />
+    <inertia ixx="${base_link_inertia_xx}" iyy="${base_link_inertia_yy}" izz="${base_link_inertia_zz}" ixy="0" ixz="0" iyz="0" />
   </inertial>
 <!--Base Link Box-->
@@ -95,6 +113,6 @@
   <inertial>
     <origin xyz="0 ${radius_small_cylinder*3/2+length_small_box*3/2+length_link1_box/2} 0" rpy="0 0 0"/>
-    <mass value="1" />
-    <inertia ixx="0.1" iyy="0.1" izz="0.1" ixy="0" ixz="0" iyz="0" />
+    <mass value="${first_link_mass}" />
+    <inertia ixx="${first_link_inertia_xx}" iyy="${first_link_inertia_yy}" izz="${first_link_inertia_zz}" ixy="0" ixz="0" iyz="0" />
   </inertial>
 <!--First Link Small Cylinder - Front -->
@@ -183,6 +201,6 @@
   <inertial>
     <origin xyz="0 ${radius_small_cylinder*3/2+length_small_box*3/2+length_link1_box/2} 0" rpy="0 0 0"/>
-    <mass value="1" />
-    <inertia ixx="0.1" iyy="0.1" izz="0.1" ixy="0" ixz="0" iyz="0" />
+    <mass value="${second_link_mass}" />
+    <inertia ixx="${second_link_inertia_xx}" iyy="${second_link_inertia_yy}" izz="${second_link_inertia_zz}" ixy="0" ixz="0" iyz="0" />
   </inertial>
 <!--Second Link Small Cylinder - Front -->
@@ -271,6 +289,6 @@
   <inertial>
     <origin xyz="0 0 ${height_base_box/4}" rpy="0 0 0"/>
-    <mass value="1" />
-    <inertia ixx="0.1" iyy="0.1" izz="0.1" ixy="0" ixz="0" iyz="0" />
+    <mass value="${handle_link_mass}"/>
+    <inertia ixx="${handle_link_inertia_xx}" iyy="${handle_link_inertia_yy}" izz="${handle_link_inertia_zz}" ixy="0" ixz="0" iyz="0" />
   </inertial>
   <visual>
@@ -326,10 +344,10 @@
   <limit effort="30" lower="-${angle}" upper="${angle}" velocity="1.0"/>
   <safety_controller k_velocity="10" k_position="15" soft_lower_limit="-1.5" soft_upper_limit="1.5"/>
-  <!--sensor name='left_leg_ft' type='force_torque'>
+  <!--sensor name='handle_ft' type='force_torque'>
     <always_on>1</always_on>
     <update_rate>100</update_rate>
     <pose>0 0 0 0 0 0</pose>
-    <plugin name='handle_ft' filename='libgazebo_yarp_forcetorque.so'>
-      <yarpConfigurationFile>model://icub/conf/FT/gazebo_forcetorque.ini</yarpConfigurationFile>
+    <plugin name='forcetorque' filename='libgazebo_yarp_forcetorque.so'>
+      <yarpConfigurationFile>model://2r_manipulator_scaled_down/conf/gazebo_forcetorque.ini</yarpConfigurationFile>
     </plugin>
   </sensor-->
