Commit message: Floating base 1RDOF removed yarp plugins

File: floating_base_1RDOF_2Link/model.urdf (robot description, URDF)
Before this commit: robot floating_base_1RDOF_2Link, 3 links, 2 joints
Joints:
- joint anchor: type floating -> fixed

File: floating_base_1RDOF_2Link/model.xacro (robot description, xacro)
@@ -12,4 +12,6 @@
 <!--XACRO: Axis Rotation - 180 Degree/ Pi Radians-->
 <xacro:property name="angle" value="3.14"/>
+<!--XACRO: Inertia Value-->
+<xacro:property name="inertia" value="0.001"/>
 <!--XACRO: Small Rectangle-->
 <xacro:property name="length_small_box" value="0.05"/>
@@ -31,15 +33,15 @@
 <xacro:property name="second_link_mass" value="1"/>
 <!--XACRO: Link Inertia Value-->
-<xacro:property name="first_link_inertia_xx" value="0.1"/>
-<xacro:property name="first_link_inertia_yy" value="0.1"/>
-<xacro:property name="first_link_inertia_zz" value="0.1"/>
-<xacro:property name="second_link_inertia_xx" value="0.1"/>
-<xacro:property name="second_link_inertia_yy" value="0.1"/>
-<xacro:property name="second_link_inertia_zz" value="0.1"/>
+<xacro:property name="first_link_inertia_xx" value="${inertia}"/>
+<xacro:property name="first_link_inertia_yy" value="${inertia}"/>
+<xacro:property name="first_link_inertia_zz" value="${inertia}"/>
+<xacro:property name="second_link_inertia_xx" value="${inertia}"/>
+<xacro:property name="second_link_inertia_yy" value="${inertia}"/>
+<xacro:property name="second_link_inertia_zz" value="${inertia}"/>
 <link name="world" />
 <!--First Link-->
 <link name="first_link">
   <inertial>
-    <origin xyz="0 0 0" rpy="0 0 0"/>
+    <origin xyz="0 ${radius_small_cylinder*3/2+length_small_box*3/2+length_link1_box/2} 0" rpy="0 0 0"/>
     <mass value="${first_link_mass}" />
     <inertia ixx="${first_link_inertia_xx}" iyy="${first_link_inertia_yy}" izz="${first_link_inertia_zz}" ixy="0" ixz="0" iyz="0" />
@@ -97,5 +99,5 @@
 <link name="second_link">
   <inertial>
-    <origin xyz="0 0 0" rpy="0 0 0"/>
+    <origin xyz="0 ${radius_small_cylinder*3/2+length_small_box*3/2+length_link2_box/2} 0" rpy="0 0 0"/>
     <mass value="${second_link_mass}" />
     <inertia ixx="${second_link_inertia_xx}" iyy="${second_link_inertia_yy}" izz="${second_link_inertia_zz}" ixy="0" ixz="0" iyz="0" />
@@ -151,5 +153,5 @@
 </link>
 <!--Joints-->
-<joint name="anchor" type="floating">
+<joint name="anchor" type="fixed">
   <parent link="world"/>
   <child link="first_link"/>
